Commit message: Did some experiment set-ups for D*Lite

File: BA_bio_inspired_navigation-main/environment/linear_sunburst_map/plane_doors_unstructured.urdf (robot description, URDF)
Before this commit: robot plane, 20 links, 19 joints
Links:
- removed link door_1
- removed link door_2
- removed link door_3
- removed link door_4
Joints:
- removed joint door_1_joint
- removed joint door_2_joint
- removed joint door_3_joint
- removed joint door_4_joint

File: BA_bio_inspired_navigation-main/environment/linear_sunburst_map/plane_unstructured.urdf (robot description, URDF)
Before this commit: robot plane, 20 links, 19 joints
Links:
- removed link door_1
- removed link door_2
- removed link door_3
- removed link door_4
Joints:
- removed joint door_1_joint
- removed joint door_2_joint
- removed joint door_3_joint
- removed joint door_4_joint
