Commit message: Experiment Setup Tested

File: BA_bio_inspired_navigation-main/environment/linear_sunburst_map/plane_unstructured_doors.urdf (robot description, URDF)
Before this commit: robot plane, 16 links, 15 joints
Links:
- added link door_1, mass 1; collision box size=1 0.2 1; visual box size=1 0.2 1
- added link door_2, mass 1; collision box size=1 0.2 1; visual box size=1 0.2 1
- added link door_3, mass 1; collision box size=1 0.2 1; visual box size=1 0.2 1
- added link door_4, mass 1; collision box size=1 0.2 1; visual box size=1 0.2 1
Joints:
- added joint door_1_joint: type fixed, parent planeLink, child door_1, origin xyz=0 0 0 rpy=0 0 0
- added joint door_2_joint: type fixed, parent planeLink, child door_2, origin xyz=0 0 0 rpy=0 0 0
- added joint door_3_joint: type fixed, parent planeLink, child door_3, origin xyz=0 0 0 rpy=0 0 0
- added joint door_4_joint: type fixed, parent planeLink, child door_4, origin xyz=0 0 0 rpy=0 0 0
